File: ATP_Teensy.kicad_sch (KiCad schematic)
At the start: 24 parts, among them J1 Screw_Terminal_01x02, J2 Conn_01x01, J3 Conn_01x01, J4 Conn_01x01, J5 Conn_01x01, J6 Conn_01x06_Male, J7 Conn_01x04_Male, U1 BMP388_3966, U2 L7805CV, U3 XBee_SparkfunRegulatedAdapter, U4 MPU6050, U5 Teensy4.1, U6 GPS

Commit message: Add labels for layout, DRC run, v1.1 Gerber files generated
Other:
- note added: "Avionics Flight Sensor (AFS)"
- note added: "Last Modified by: Alexandra Zhang Jiang on MAR 06th, 2023"
- note removed: "Avionics Test Payload (ATP)"
- note removed: "Last Modified by: Alexandra Zhang Jiang on DEC 18th, 2022"
- moved on the sheet: C3, C4, C5
